File: Schematics/Car LED Controller Schematic V4 - KiCAD/Car LED Controller Schematic V4 - KiCAD.kicad_pcb (KiCad board)
At the start: 2 copper layers, 101.9 x 70 mm, 20 parts, among them J1 5V Power In, J2 Select Button, J3 LCD, Relay, LED Signal, J4 ZSS-108-01-F-D-506, J5 Conn_01x05_Pin, U1 ESP32-DEVKITC-32D, U2 BOB-12009

Commit message: more pcb designs
Parts:
- J1, J2: footprint Connector_PinHeader_2.54mm:PinHeader_1x02_P2.54mm_Vertical -> Connector_JST:JST_XH_B2B-XH-A_1x02_P2.50mm_Vertical
- J3: footprint Connector_PinHeader_2.54mm:PinHeader_1x06_P2.54mm_Vertical -> Connector_JST:JST_XH_B6B-XH-A_1x06_P2.50mm_Vertical
- J5: value Conn_01x05_Pin -> DRL, Horn Sense; footprint Connector_PinHeader_2.54mm:PinHeader_1x05_P2.54mm_Vertical -> Connector_JST:JST_XH_B5B-XH-A_1x05_P2.50mm_Vertical
- moved R12 64.2 mm to (67.0, 83.5)
- moved R13 60.5 mm to (67.0, 80.4), turned to 0 degrees
- moved J3 59.5 mm to (62.3, 89.2), turned to 180 degrees
- moved R11 59.4 mm to (124.7, 87.5), turned to 180 degrees
- moved R10 59.2 mm to (127.4, 87.6), turned to 90 degrees
- moved J2 58.8 mm to (47.2, 44.1)
- moved J1 56.8 mm to (48.1, 30.1), turned to -90 degrees
- moved C5 56.6 mm to (124.7, 84.3)
- moved C6 55.8 mm to (66.9, 76.9), turned to 0 degrees
- moved U2 48.2 mm to (56.1, 70.5)
- moved C8 45.8 mm to (124.9, 25.8), turned to -90 degrees
- moved R17 43.9 mm to (121.8, 25.8)
- moved R16 43.3 mm to (118.7, 25.8), turned to -90 degrees
- moved C7 42.4 mm to (69.2, 63.5), turned to -90 degrees
- moved R15 41.6 mm to (72.3, 58.3)
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Connections:
- J5 pad 1: GND -> Net-(J5-Pin_1)
- J5 pad 5: Net-(J5-Pin_5) -> GND
- R10 pad 2: Net-(J5-Pin_5) -> Net-(J5-Pin_1)
- R12 pad 2: Net-(J5-Pin_4) -> Net-(J5-Pin_2)
- R16 pad 2: Net-(J5-Pin_2) -> Net-(J5-Pin_4)
- U1 pad J3-10: Net-(J4-LAT) -> Net-(J4-G1)
- U1 pad J3-11: Net-(J4-D) -> Net-(J4-G2)
- U1 pad J3-12: Net-(J4-B) -> Net-(J4-E)
- U1 pad J3-13: Net-(J4-E) -> Net-(J4-B)
- U1 pad J3-15: Net-(J4-G2) -> Net-(J4-D)
- U1 pad J3-16: Net-(J4-G1) -> Net-(J4-LAT)
Routing:
- net GND: track 264.8 -> 350.9 mm
- net Net-(J5-Pin_2): track 14.0 -> 81.1 mm
- net Net-(U1-SENSOR_VP): track 28.6 -> 93.1 mm, vias 0 -> 1
- net Net-(J5-Pin_3): track 24.6 -> 87.2 mm
- net Net-(J4-LAT): track 23.5 -> 70.1 mm
- net Net-(J5-Pin_5): track 45.8 -> 0.00 mm
- net Net-(J4-B): track 23.5 -> 67.6 mm
- net Net-(J4-D): track 23.5 -> 67.4 mm
- net Net-(J4-E): track 23.5 -> 65.1 mm
- net +3.3V: track 56.4 -> 15.3 mm
- net Net-(J4-G2): track 24.4 -> 62.8 mm
- net Net-(J4-R1): track 51.4 -> 13.3 mm
- net Net-(J4-B1): track 55.7 -> 17.9 mm
- net Net-(J4-G1): track 23.5 -> 59.2 mm
- net Net-(J4-R2): track 56.4 -> 21.5 mm
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Other:
- board text removed: "RESET - EN"
