File: Schematics/Control Board Yves/Control Board.kicad_pcb (KiCad board)
At the start: 2 copper layers, 101.9 x 70 mm, 20 parts, among them J1 5V Power In, J2 Select Button, J3 LCD, Relay, LED Signal, J4 ZSS-108-01-F-D-506, J5 Conn_01x05_Pin, U1 ESP32-DEVKITC-32D, U2 BOB-12009

Commit message: cleanup of pcb
Routing:
- net GND: track 337.9 -> 323.0 mm
- net Net-(J2-Pin_1): track 129.1 -> 114.9 mm
- net Net-(J4-G2): track 81.0 -> 71.5 mm
- net Net-(U1-SENSOR_VP): track 111.0 -> 101.7 mm
- net Net-(J4-B): track 98.0 -> 88.9 mm
- net +5V: track 181.1 -> 172.5 mm
- net Net-(J4-E): track 92.7 -> 84.1 mm
- net Net-(U1-SENSOR_VN): track 104.9 -> 96.5 mm
- net Net-(J4-D): track 119.5 -> 111.2 mm
- net Net-(J4-LAT): track 131.3 -> 123.9 mm
- net Net-(J4-G1): track 62.6 -> 55.7 mm
- net Net-(U1-IO35): track 92.3 -> 85.5 mm
- net Net-(U1-IO23): track 45.5 -> 39.3 mm
- net Net-(J3-Pin_4): track 96.9 -> 91.5 mm
- net Net-(J3-Pin_2): track 113.3 -> 108.5 mm
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Other:
- outline, holes or cut-outs redrawn
- board text added: "LED Matrix Controller V3"
- board text removed: "LED Matrix Controller V1"

Commit message: more pcb designs
Parts:
- J1, J2: footprint Connector_PinHeader_2.54mm:PinHeader_1x02_P2.54mm_Vertical -> Connector_JST:JST_XH_B2B-XH-A_1x02_P2.50mm_Vertical
- J3: footprint Connector_PinHeader_2.54mm:PinHeader_1x06_P2.54mm_Vertical -> Connector_JST:JST_XH_B6B-XH-A_1x06_P2.50mm_Vertical
- moved J2 60.3 mm to (116.0, 65.1), turned to 0 degrees
- moved J1 1.86 mm to (48.5, 89.6), turned to 0 degrees
- moved J3 1.54 mm to (50.2, 83.0), turned to 90 degrees
- renumbered R10 to R1
Routing:
- net Net-(J2-Pin_1): track 114.9 -> 14.9 mm, vias 1 -> 0
- net GND: track 323.0 -> 313.5 mm
- net Net-(U1-SENSOR_VP): track 101.7 -> 95.5 mm
- net Net-(U1-SENSOR_VN): track 96.5 -> 90.6 mm
- net Net-(J3-Pin_2): track 108.5 -> 110.0 mm
- net Net-(U1-IO19): track 26.9 -> 28.3 mm
- net Net-(U1-IO35): track 85.5 -> 86.8 mm
- net +5V: track 172.5 -> 173.7 mm
- net Net-(J4-OE): track 16.0 -> 14.8 mm
- net Net-(J3-Pin_3): track 102.7 -> 103.6 mm
- net Net-(J3-Pin_5): track 84.4 -> 83.9 mm
