File: Schematics/Car LED Controller Schematic V8 - KiCAD/Car LED Controller Schematic V8 - KiCAD.kicad_sch (KiCad schematic)
At the start: 20 parts, among them J2 LCD, Relay, LED Signal, J3 5V Power In, J4 Select Button, J4 ZSS-108-01-F-D-506, J5 DRL, Horn Sense, U1 ESP32-DEVKITC-32D, U2 BOB-12009

Commit message: more pcb designs
Connections:
- net at J4.01 (R1): now also U1.J2-7 (IO32); no longer U1.J2-15 (IO13)
- net Net-(J4-G1): now reaches U1.J3-10 (IO5)
- net Net-(J4-G1): now also J4.14 (LAT); no longer J4.02 (G1)
- net at J4.03 (B1): now also U1.J2-8 (IO33); no longer U1.J2-13 (IO12)
- net at J4.05 (R2): now also U1.J2-9 (IO25); no longer U1.J2-12 (IO14)
- net Net-(J4-D): now reaches J4.06 (G2)
- net Net-(J4-D): now also U1.J3-15 (IO2); no longer U1.J3-11 (IO17)
- net at J4.07 (B2): now also U1.J2-10 (IO26); no longer U1.J2-11 (IO27)
- net Net-(J4-B): now reaches J4.08 (E)
- net Net-(J4-B): now also U1.J3-13 (IO4); no longer U1.J3-12 (IO16)
- net at J4.09 (A): now also U1.J2-11 (IO27); no longer U1.J2-10 (IO26)
- net Net-(J4-E): now reaches J4.10 (B)
- net Net-(J4-E): now also U1.J3-12 (IO16); no longer U1.J3-13 (IO4)
- net at J4.11 (C): now also U1.J2-12 (IO14); no longer U1.J2-9 (IO25)
- net Net-(J4-G2): now reaches J4.12 (D)
- net Net-(J4-G2): now also U1.J3-11 (IO17); no longer U1.J3-15 (IO2)
- net at J4.13 (CLK): now also U1.J2-13 (IO12); no longer U1.J2-8 (IO33)
- net Net-(J4-LAT): now reaches U1.J3-16 (IO15)
- net Net-(J4-LAT): now also J4.02 (G1); no longer J4.14 (LAT)
- net at J4.15 (OE): now also U1.J2-15 (IO13); no longer U1.J2-7 (IO32)
Changed lines of the file:
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@@
   (junction (at 233.68 88.9) (diameter 0) (color 0 0 0 0)
   )
-  (wire (pts (xy 62.23 74.93) (xy 120.65 74.93))
-    (stroke (width 0) (type default))
-  )
-  (wire (pts (xy 52.07 64.77) (xy 130.81 64.77))
+  (wire (pts (xy 54.61 74.93) (xy 120.65 74.93))
     (stroke (width 0) (type default))
   )
@@
     (stroke (width 0) (type default))
   )
+  (wire (pts (xy 62.23 67.31) (xy 62.23 88.9))
+    (stroke (width 0) (type default))
+  )
   (wire (pts (xy 125.73 138.43) (xy 125.73 166.37))
     (stroke (width 0) (type default))
@@
     (stroke (width 0) (type default))
   )
+  (wire (pts (xy 59.69 69.85) (xy 125.73 69.85))
+    (stroke (width 0) (type default))
+  )
   (wire (pts (xy 228.6 60.96) (xy 153.67 60.96))
     (stroke (width 0) (type default))
@@
     (stroke (width 0) (type default))
   )
+  (wire (pts (xy 62.23 114.3) (xy 62.23 156.21))
+    (stroke (width 0) (type default))
+  )
   (wire (pts (xy 213.36 36.83) (xy 210.82 36.83))
     (stroke (width 0) (type default))
   )
-  (wire (pts (xy 57.15 69.85) (xy 125.73 69.85))
+  (wire (pts (xy 64.77 64.77) (xy 64.77 88.9))
     (stroke (width 0) (type default))
   )
@@
     (stroke (width 0) (type default))
   )
-  (wire (pts (xy 67.31 88.9) (xy 67.31 80.01))
-    (stroke (width 0) (type default))
-  )
-  (wire (pts (xy 62.23 163.83) (xy 62.23 114.3))
-    (stroke (width 0) (type default))
-  )
   (wire (pts (xy 135.89 157.48) (xy 190.5 157.48))
     (stroke (width 0) (type default))
   )
-  (wire (pts (xy 118.11 158.75) (xy 57.15 158.75))
+  (wire (pts (xy 118.11 158.75) (xy 59.69 158.75))
     (stroke (width 0) (type default))
   )
@@
     (stroke (width 0) (type default))
   )
+  (wire (pts (xy 62.23 156.21) (xy 113.03 156.21))
+    (stroke (width 0) (type default))
+  )
   (wire (pts (xy 120.65 74.93) (xy 120.65 97.79))
     (stroke (width 0) (type default))
   )
-  (wire (pts (xy 54.61 156.21) (xy 54.61 114.3))
-    (stroke (width 0) (type default))
-  )
   (wire (pts (xy 86.36 87.63) (xy 115.57 87.63))
     (stroke (width 0) (type default))
   )
+  (wire (pts (xy 57.15 72.39) (xy 57.15 88.9))
+    (stroke (width 0) (type default))
+  )
+  (wire (pts (xy 54.61 114.3) (xy 54.61 163.83))
+    (stroke (width 0) (type default))
+  )
   (wire (pts (xy 125.73 97.79) (xy 125.73 69.85))
     (stroke (width 0) (type default))
   )
-  (wire (pts (xy 110.49 153.67) (xy 52.07 153.67))
-    (stroke (width 0) (type default))
-  )
   (wire (pts (xy 113.03 138.43) (xy 113.03 156.21))
     (stroke (width 0) (type default))
@@
     (stroke (width 0) (type default))
   )
-  (wire (pts (xy 67.31 166.37) (xy 67.31 114.3))
-    (stroke (width 0) (type default))
-  )
-  (wire (pts (xy 123.19 163.83) (xy 62.23 163.83))
-    (stroke (width 0) (type default))
-  )
-  (wire (pts (xy 67.31 80.01) (xy 113.03 80.01))
+  (wire (pts (xy 67.31 62.23) (xy 133.35 62.23))
+    (stroke (width 0) (type default))
+  )
+  (wire (pts (xy 54.61 163.83) (xy 123.19 163.83))
+    (stroke (width 0) (type default))
+  )
+  (wire (pts (xy 52.07 166.37) (xy 125.73 166.37))
+    (stroke (width 0) (type default))
+  )
+  (wire (pts (xy 49.53 80.01) (xy 113.03 80.01))
     (stroke (width 0) (type default))
   )
@@
     (stroke (width 0) (type default))
   )
-  (wire (pts (xy 120.65 161.29) (xy 59.69 161.29))
+  (wire (pts (xy 57.15 161.29) (xy 120.65 161.29))
     (stroke (width 0) (type default))
   )
@@
     (stroke (width 0) (type default))
   )
+  (wire (pts (xy 67.31 153.67) (xy 67.31 114.3))
+    (stroke (width 0) (type default))
+  )
   (wire (pts (xy 130.81 138.43) (xy 130.81 146.05))
     (stroke (width 0) (type default))
@@
     (stroke (width 0) (type default))
   )
-  (wire (pts (xy 62.23 88.9) (xy 62.23 74.93))
-    (stroke (width 0) (type default))
-  )
-  (wire (pts (xy 59.69 88.9) (xy 59.69 72.39))
+  (wire (pts (xy 52.07 114.3) (xy 52.07 166.37))
     (stroke (width 0) (type default))
   )
@@
     (stroke (width 0) (type default))
   )
-  (wire (pts (xy 54.61 88.9) (xy 54.61 67.31))
-    (stroke (width 0) (type default))
-  )
   (wire (pts (xy 135.89 97.79) (xy 135.89 62.23))
     (stroke (width 0) (type default))
@@
     (stroke (width 0) (type default))
   )
+  (wire (pts (xy 52.07 77.47) (xy 52.07 88.9))
+    (stroke (width 0) (type default))
+  )
   (wire (pts (xy 172.72 88.9) (xy 172.72 91.44))
     (stroke (width 0) (type default))
   )
+  (wire (pts (xy 110.49 153.67) (xy 67.31 153.67))
+    (stroke (width 0) (type default))
+  )
   (wire (pts (xy 241.3 72.39) (xy 213.36 72.39))
     (stroke (width 0) (type default))
   )
-  (wire (pts (xy 59.69 161.29) (xy 59.69 114.3))
+  (wire (pts (xy 62.23 67.31) (xy 128.27 67.31))
     (stroke (width 0) (type default))
   )
@@
     (stroke (width 0) (type default))
   )
-  (wire (pts (xy 59.69 72.39) (xy 123.19 72.39))
+  (wire (pts (xy 57.15 72.39) (xy 123.19 72.39))
     (stroke (width 0) (type default))
   )
@@
     (stroke (width 0) (type default))
   )
+  (wire (pts (xy 54.61 74.93) (xy 54.61 88.9))
+    (stroke (width 0) (type default))
+  )
   (wire (pts (xy 187.96 91.44) (xy 187.96 88.9))
     (stroke (width 0) (type default))
@@
     (stroke (width 0) (type default))
   )
+  (wire (pts (xy 59.69 69.85) (xy 59.69 88.9))
+    (stroke (width 0) (type default))
+  )
   (wire (pts (xy 233.68 88.9) (xy 233.68 91.44))
     (stroke (width 0) (type default))
@@
     (stroke (width 0) (type default))
   )
-  (wire (pts (xy 52.07 153.67) (xy 52.07 114.3))
+  (wire (pts (xy 57.15 114.3) (xy 57.15 161.29))
+    (stroke (width 0) (type default))
+  )
+  (wire (pts (xy 64.77 64.77) (xy 130.81 64.77))
     (stroke (width 0) (type default))
   )
@@
     (stroke (width 0) (type default))
   )
+  (wire (pts (xy 59.69 114.3) (xy 59.69 158.75))
+    (stroke (width 0) (type default))
+  )
   (wire (pts (xy 241.3 67.31) (xy 172.72 67.31))
     (stroke (width 0) (type default))
   )
+  (wire (pts (xy 67.31 62.23) (xy 67.31 88.9))
+    (stroke (width 0) (type default))
+  )
   (wire (pts (xy 208.28 62.23) (xy 208.28 88.9))
     (stroke (width 0) (type default))
@@
     (stroke (width 0) (type default))
   )
-  (wire (pts (xy 64.77 77.47) (xy 118.11 77.47))
+  (wire (pts (xy 52.07 77.47) (xy 118.11 77.47))
     (stroke (width 0) (type default))
   )
@@
     (stroke (width 0) (type default))
   )
-  (wire (pts (xy 54.61 67.31) (xy 128.27 67.31))
-    (stroke (width 0) (type default))
-  )
-  (wire (pts (xy 49.53 62.23) (xy 133.35 62.23))
-    (stroke (width 0) (type default))
-  )
   (wire (pts (xy 133.35 62.23) (xy 133.35 97.79))
     (stroke (width 0) (type default))
@@
     (stroke (width 0) (type default))
   )
-  (wire (pts (xy 57.15 88.9) (xy 57.15 69.85))
-    (stroke (width 0) (type default))
-  )
-  (wire (pts (xy 125.73 166.37) (xy 67.31 166.37))
-    (stroke (width 0) (type default))
-  )
   (wire (pts (xy 146.05 152.4) (xy 190.5 152.4))
     (stroke (width 0) (type default))
   )
-  (wire (pts (xy 113.03 156.21) (xy 54.61 156.21))
+  (wire (pts (xy 49.53 80.01) (xy 49.53 88.9))
     (stroke (width 0) (type default))
   )
@@
     (stroke (width 0) (type default))
   )
-  (wire (pts (xy 64.77 77.47) (xy 64.77 88.9))
-    (stroke (width 0) (type default))
-  )
-  (wire (pts (xy 57.15 158.75) (xy 57.15 114.3))
-    (stroke (width 0) (type default))
-  )
-  (wire (pts (xy 49.53 62.23) (xy 49.53 88.9))
-    (stroke (width 0) (type default))
-  )
   (wire (pts (xy 120.65 138.43) (xy 120.65 161.29))
     (stroke (width 0) (type default))
@@
     (stroke (width 0) (type default))
   )
-  (wire (pts (xy 52.07 88.9) (xy 52.07 64.77))
-    (stroke (width 0) (type default))
+  (label "Net-(J4-E)" (at 57.15 114.3 270)
+    (effects (font (size 1.27 1.27)) (justify right bottom))
+  )
+  (label "Net-(J4-D)" (at 62.23 114.3 270)
+    (effects (font (size 1.27 1.27)) (justify right bottom))
+  )
+  (label "Net-(J4-LAT)" (at 67.31 114.3 270)
+    (effects (font (size 1.27 1.27)) (justify right bottom))
+  )
+  (label "Net-(J4-B)" (at 59.69 114.3 270)
+    (effects (font (size 1.27 1.27)) (justify right bottom))
+  )
+  (label "Net-(J4-G2)" (at 54.61 114.3 270)
+    (effects (font (size 1.27 1.27)) (justify right bottom))
+  )
+  (label "Net-(J4-G1)" (at 52.07 114.3 270)
+    (effects (font (size 1.27 1.27)) (justify right bottom))
   )
   (symbol (lib_id "power:GND") (at 86.36 87.63 0) (unit 1)

Commit message: more pcb
Connections:
- net at J4.01 (R1): now also U1.J2-9 (IO25); no longer U1.J2-7 (IO32)
- net at J4.05 (R2): now also U1.J2-12 (IO14); no longer U1.J2-9 (IO25)
- net at U1.J2-10 (IO26): now also J4.02 (G1); no longer J4.07 (B2)
- net at J4.11 (C): now also U1.J3-10 (IO5); no longer U1.J2-12 (IO14)
- net at U1.J2-13 (IO12): now also J4.06 (G2); no longer J4.13 (CLK)
- net at U1.J2-15 (IO13): now also J4.07 (B2); no longer J4.15 (OE)
- net Net-(J4-B): no longer names the net of J4.08 (E)
- net Net-(J4-B): now also U1.J2-7 (IO32); no longer U1.J3-13 (IO4)
- net Net-(J4-D): no longer names the net of U1.J3-15 (IO2)
- net Net-(J4-D): now also J4.10 (B); no longer J4.06 (G2)
- net Net-(J4-E): no longer names the net of U1.J3-12 (IO16)
- net Net-(J4-E): now also J4.13 (CLK); no longer J4.10 (B)
- net Net-(J4-G1): no longer names the net of J4.14 (LAT)
- net Net-(J4-G1): now also U1.J3-13 (IO4); no longer U1.J3-10 (IO5)
- net Net-(J4-G2): no longer names the net of J4.12 (D), U1.J3-11 (IO17)
- net Net-(J4-LAT): no longer names the net of U1.J3-16 (IO15)
- net Net-(J4-LAT): now also J4.15 (OE); no longer J4.02 (G1)

Commit message: added more details
Connections:
- net GND: now also J5.Res (Pin_5); no longer J5.5 (Pin_5)
- net at U2.HV1: now also J2.LED (Pin_2); no longer J2.2 (Pin_2)
- net at U2.HV2: now also J2.Relay (Pin_3); no longer J2.3 (Pin_3)
- net at U2.HV3: now also J2.LCD (Pin_5); no longer J2.4 (Pin_4)
- net at U2.HV4: now also J2.LCD (Pin_5); no longer J2.5 (Pin_5)
- net at R9.2: now also J5.DRL (Pin_2); no longer J5.2 (Pin_2)
- net at R9.2: now also J5.Horn (Pin_3); no longer J5.3 (Pin_3)
- net at R9.2: now also J5.Res (Pin_5); no longer J5.4 (Pin_4)
Other:
- moved on the sheet: J2
Changed lines of the file:
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@@
     )
     (pin "1")
-    (pin "2")
-    (pin "3")
-    (pin "4")
-    (pin "5")
+    (pin "DRL")
+    (pin "Horn")
+    (pin "Res")
+    (pin "Res")
     (instances
       (project "Car LED Controller Schematic V8 - KiCAD"
@@
     )
     (pin "1")
-    (pin "2")
-    (pin "3")
-    (pin "4")
-    (pin "5")
+    (pin "LED")
+    (pin "Relay")
+    (pin "LCD")
+    (pin "LCD")
     (pin "6")
     (instances

Commit message: updated Schematic
Parts:
- added J4: Reset Button, Connector_JST:JST_XH_B2B-XH-A_1x02_P2.50mm_Vertical, symbol Connector_Generic:Conn_01x02
Connections:
- net GND: now also J4.2 (Pin_2)
- net at U1.J2-2 (EN): now also J4.1 (Pin_1)
Other:
- moved on the sheet: J4, R1
Changed lines of the file:
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@@
   (junction (at 187.96 88.9) (diameter 0) (color 0 0 0 0)
   )
-  (junction (at 153.67 39.37) (diameter 0) (color 0 0 0 0)
+  (junction (at 153.67 33.02) (diameter 0) (color 0 0 0 0)
   )
   (junction (at 172.72 88.9) (diameter 0) (color 0 0 0 0)
@@
     (stroke (width 0) (type default))
   )
-  (wire (pts (xy 138.43 39.37) (xy 153.67 39.37))
+  (wire (pts (xy 146.05 49.53) (xy 146.05 97.79))
+    (stroke (width 0) (type default))
+  )
+  (wire (pts (xy 138.43 33.02) (xy 153.67 33.02))
     (stroke (width 0) (type default))
   )
@@
     (stroke (width 0) (type default))
   )
-  (wire (pts (xy 153.67 35.56) (xy 153.67 39.37))
+  (wire (pts (xy 153.67 29.21) (xy 153.67 33.02))
     (stroke (width 0) (type default))
   )
@@
     (stroke (width 0) (type default))
   )
-  (wire (pts (xy 138.43 39.37) (xy 138.43 97.79))
+  (wire (pts (xy 138.43 33.02) (xy 138.43 97.79))
     (stroke (width 0) (type default))
   )
@@
     (stroke (width 0) (type default))
   )
+  (wire (pts (xy 146.05 49.53) (xy 153.67 49.53))
+    (stroke (width 0) (type default))
+  )
   (wire (pts (xy 96.52 92.71) (xy 96.52 118.11))
     (stroke (width 0) (type default))
@@
         (path "/a58fb6f5-162c-4767-8872-78e5b371198c"
           (reference "#PWR021") (unit 1)
+        )
+      )
+    )
+  )
+  (symbol (lib_id "Connector_Generic:Conn_01x02") (at 158.75 49.53 0) (unit 1)
+    (in_bom yes) (on_board yes) (dnp no)
+    (property "Reference" "J4" (at 165.1 55.88 90)
+      (effects (font (size 1.27 1.27)) (justify left))
+    )
+    (property "Value" "Reset Button" (at 162.56 55.88 90)
+      (effects (font (size 1.27 1.27)) (justify left))
+    )
+    (property "Footprint" "Connector_JST:JST_XH_B2B-XH-A_1x02_P2.50mm_Vertical" (at 158.75 49.53 0)
+      (effects (font (size 1.27 1.27)) hide)
+    )
+    (property "Datasheet" "~" (at 158.75 49.53 0)
+      (effects (font (size 1.27 1.27)) hide)
+    )
+    (pin "1")
+    (pin "2")
+    (instances
+      (project "Car LED Controller"
+        (path "/343b98cc-35d9-4f95-bcfd-36dc76d2ef8d"
+          (reference "J4") (unit 1)
+        )
+      )
+      (project "Car LED Controller Schematic V8 - KiCAD"
+        (path "/a58fb6f5-162c-4767-8872-78e5b371198c"
+          (reference "J6") (unit 1)
         )
       )
@@
     )
   )
-  (symbol (lib_id "Connector_Generic:Conn_01x02") (at 158.75 39.37 0) (unit 1)
-    (in_bom yes) (on_board yes) (dnp no)
-    (property "Reference" "J4" (at 165.1 45.72 90)
+  (symbol (lib_id "Connector_Generic:Conn_01x02") (at 158.75 33.02 0) (unit 1)
+    (in_bom yes) (on_board yes) (dnp no)
+    (property "Reference" "J4" (at 165.1 39.37 90)
       (effects (font (size 1.27 1.27)) (justify left))
     )
-    (property "Value" "Select Button" (at 162.56 45.72 90)
+    (property "Value" "Select Button" (at 162.56 39.37 90)
       (effects (font (size 1.27 1.27)) (justify left))
     )
-    (property "Footprint" "Connector_JST:JST_XH_B2B-XH-A_1x02_P2.50mm_Vertical" (at 158.75 39.37 0)
-      (effects (font (size 1.27 1.27)) hide)
-    )
-    (property "Datasheet" "~" (at 158.75 39.37 0)
+    (property "Footprint" "Connector_JST:JST_XH_B2B-XH-A_1x02_P2.50mm_Vertical" (at 158.75 33.02 0)
+      (effects (font (size 1.27 1.27)) hide)
+    )
+    (property "Datasheet" "~" (at 158.75 33.02 0)
       (effects (font (size 1.27 1.27)) hide)
     )
@@
     )
   )
-  (symbol (lib_id "power:+3.3V") (at 153.67 27.94 0) (unit 1)
-    (in_bom yes) (on_board yes) (dnp no) (fields_autoplaced)
-    (property "Reference" "#PWR026" (at 153.67 31.75 0)
-      (effects (font (size 1.27 1.27)) hide)
-    )
-    (property "Value" "+3.3V" (at 153.67 24.13 0)
-      (effects (font (size 1.27 1.27)))
-    )
-    (property "Footprint" "" (at 153.67 27.94 0)
-      (effects (font (size 1.27 1.27)) hide)
-    )
-    (property "Datasheet" "" (at 153.67 27.94 0)
+  (symbol (lib_id "power:+3.3V") (at 153.67 21.59 0) (unit 1)
+    (in_bom yes) (on_board yes) (dnp no) (fields_autoplaced)
+    (property "Reference" "#PWR026" (at 153.67 25.4 0)
+      (effects (font (size 1.27 1.27)) hide)
+    )
+    (property "Value" "+3.3V" (at 153.67 17.78 0)
+      (effects (font (size 1.27 1.27)))
+    )
+    (property "Footprint" "" (at 153.67 21.59 0)
+      (effects (font (size 1.27 1.27)) hide)
+    )
+    (property "Datasheet" "" (at 153.67 21.59 0)
       (effects (font (size 1.27 1.27)) hide)
     )
@@
     )
   )
-  (symbol (lib_id "power:GND") (at 153.67 41.91 0) (unit 1)
-    (in_bom yes) (on_board yes) (dnp no) (fields_autoplaced)
-    (property "Reference" "#PWR013" (at 153.67 48.26 0)
-      (effects (font (size 1.27 1.27)) hide)
-    )
-    (property "Value" "GND" (at 153.67 46.99 0)
-      (effects (font (size 1.27 1.27)))
-    )
-    (property "Footprint" "" (at 153.67 41.91 0)
-      (effects (font (size 1.27 1.27)) hide)
-    )
-    (property "Datasheet" "" (at 153.67 41.91 0)
+  (symbol (lib_id "power:GND") (at 153.67 52.07 0) (unit 1)
+    (in_bom yes) (on_board yes) (dnp no) (fields_autoplaced)
+    (property "Reference" "#PWR016" (at 153.67 58.42 0)
+      (effects (font (size 1.27 1.27)) hide)
+    )
+    (property "Value" "GND" (at 153.67 57.15 0)
+      (effects (font (size 1.27 1.27)))
+    )
+    (property "Footprint" "" (at 153.67 52.07 0)
+      (effects (font (size 1.27 1.27)) hide)
+    )
+    (property "Datasheet" "" (at 153.67 52.07 0)
+      (effects (font (size 1.27 1.27)) hide)
+    )
+    (pin "1")
+    (instances
+      (project "Car LED Controller Schematic V8 - KiCAD"
+        (path "/a58fb6f5-162c-4767-8872-78e5b371198c"
+          (reference "#PWR016") (unit 1)
+        )
+      )
+    )
+  )
+  (symbol (lib_id "power:GND") (at 153.67 35.56 0) (unit 1)
+    (in_bom yes) (on_board yes) (dnp no) (fields_autoplaced)
+    (property "Reference" "#PWR013" (at 153.67 41.91 0)
+      (effects (font (size 1.27 1.27)) hide)
+    )
+    (property "Value" "GND" (at 153.67 40.64 0)
+      (effects (font (size 1.27 1.27)))
+    )
+    (property "Footprint" "" (at 153.67 35.56 0)
+      (effects (font (size 1.27 1.27)) hide)
+    )
+    (property "Datasheet" "" (at 153.67 35.56 0)
       (effects (font (size 1.27 1.27)) hide)
     )
@@
     )
   )
-  (symbol (lib_id "Device:R") (at 153.67 31.75 0) (unit 1)
-    (in_bom yes) (on_board yes) (dnp no)
-    (property "Reference" "R1" (at 154.94 30.48 0)
+  (symbol (lib_id "Device:R") (at 153.67 25.4 0) (unit 1)
+    (in_bom yes) (on_board yes) (dnp no)
+    (property "Reference" "R1" (at 154.94 24.13 0)
       (effects (font (size 1.27 1.27)) (justify left))
     )
-    (property "Value" "1M" (at 154.94 33.02 0)
+    (property "Value" "1M" (at 154.94 26.67 0)
       (effects (font (size 1.27 1.27)) (justify left))
     )
-    (property "Footprint" "Resistor_THT:R_Axial_DIN0207_L6.3mm_D2.5mm_P10.16mm_Horizontal" (at 151.892 31.75 90)
-      (effects (font (size 1.27 1.27)) hide)
-    )
-    (property "Datasheet" "~" (at 153.67 31.75 0)
-      (effects (font (size 1.27 1.27)) hide)
-    )
+    (property "Footprint" "Resistor_THT:R_Axial_DIN0207_L6.3mm_D2.5mm_P10.16mm_Horizontal" (at 151.892 25.4 90)
+      (effects (font (size 1.27 1.27)) hide)
+    )
+    (property "Datasheet" "~" (at 153.67 25.4 0)
+      (effects (font (size 1.27 1.27)) hide)
+    )

Commit message: update schmetic and pcb
Connections:
- net GND: now also J5.5 (GND); no longer J5.Res (Pin_5)
- net at U2.HV1: now also J2.2 (LED); no longer J2.LED (Pin_2)
- net at U2.HV2: now also J2.3 (Relay); no longer J2.Relay (Pin_3)
- net at U2.HV3: now also J2.4 (LCD); no longer J2.LCD (Pin_5)
- net at U2.HV4: now also J2.5 (LCD); no longer J2.LCD (Pin_5)
- net at R9.2: now also J5.2 (Horn); no longer J5.DRL (Pin_2)
- net at R9.2: now also J5.3 (Res); no longer J5.Horn (Pin_3)
- net at R9.2: now also J5.4 (Res); no longer J5.Res (Pin_5)
Changed lines of the file:
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@@
       (effects (font (size 1.27 1.27)) (justify left))
     )
-    (property "Value" "DRL, Horn Sense" (at 248.92 82.55 90)
+    (property "Value" "DRL, Horn Sense" (at 252.73 82.55 90)
       (effects (font (size 1.27 1.27)) (justify left))
     )
@@
     )
     (pin "1")
-    (pin "DRL")
-    (pin "Horn")
-    (pin "Res")
-    (pin "Res")
+    (pin "2")
+    (pin "3")
+    (pin "4")
+    (pin "5")
     (instances
       (project "Car LED Controller Schematic V8 - KiCAD"
@@
   (symbol (lib_id "Connector_Generic:Conn_01x06") (at 241.3 152.4 0) (unit 1)
     (in_bom yes) (on_board yes) (dnp no)
-    (property "Reference" "J2" (at 247.65 160.02 90)
-      (effects (font (size 1.27 1.27)) (justify left))
-    )
-    (property "Value" "LCD, Relay, LED Signal" (at 245.11 160.02 90)
+    (property "Reference" "J2" (at 251.46 161.29 90)
+      (effects (font (size 1.27 1.27)) (justify left))
+    )
+    (property "Value" "LCD, Relay, LED Signal" (at 248.92 161.29 90)
       (effects (font (size 1.27 1.27)) (justify left))
     )
@@
     )
     (pin "1")
-    (pin "LED")
-    (pin "Relay")
-    (pin "LCD")
-    (pin "LCD")
+    (pin "2")
+    (pin "3")
+    (pin "4")
+    (pin "5")
     (pin "6")
     (instances
