File: Schematics/Car LED Controller Schematic V8 - KiCAD/_autosave-Car LED Controller Schematic V8 - KiCAD.kicad_pcb (KiCad board)
At the start: 2 copper layers, 101.9 x 70 mm, 21 parts, among them J1 5V Power In, J2 Select Button, J3 LCD, Relay, LED Signal, J4 ZSS-108-01-F-D-506, J5 DRL, Horn Sense, J6 Reset Button, U1 ESP32-DEVKITC-32D, U2 BOB-12009

Commit message: update schmetic and pcb
Changed lines of the file:
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@@
     (fp_line (start 14.95 3.4) (end 14.95 -2.35)
       (stroke (width 0.1) (type solid)) (layer "F.Fab"))
-    (pad "1" thru_hole roundrect (at 0 0) (size 1.7 1.95) (drill 0.95) (layers "*.Cu" "*.Mask") (roundrect_rratio 0.147059)
+    (pad "1" thru_hole roundrect (at 0 0) (size 1.7 1.95) (drill 0.95) (layers "*.Cu" "*.Mask") (roundrect_rratio 0.1470588235)
       (net 6 "+5V") (pinfunction "+5V") (pintype "passive"))
     (pad "2" thru_hole oval (at 2.5 0) (size 1.7 1.95) (drill 0.95) (layers "*.Cu" "*.Mask")
@@
     (fp_line (start 4.95 3.4) (end 4.95 -2.35)
       (stroke (width 0.1) (type solid)) (layer "F.Fab"))
-    (pad "1" thru_hole roundrect (at 0 0 90) (size 1.7 2) (drill 1) (layers "*.Cu" "*.Mask") (roundrect_rratio 0.147059)
+    (pad "1" thru_hole roundrect (at 0 0 90) (size 1.7 2) (drill 1) (layers "*.Cu" "*.Mask") (roundrect_rratio 0.1470588235)
       (net 19 "Net-(J6-Pin_1)") (pinfunction "Pin_1") (pintype "passive"))
     (pad "2" thru_hole oval (at 2.5 0 90) (size 1.7 2) (drill 1) (layers "*.Cu" "*.Mask")
