File: Schematics/Car LED Controller V2 - Jim/Car LED Controller V2 - Jim.kicad_pcb (KiCad board)
At the start: 2 copper layers, 100 x 95 mm, 2 parts

Commit message: added more details
Parts:
- added REF**: SAMTEC_FHP-04-01-X-S, Library:SAMTEC_FHP-04-01-X-S, F.Cu at (141.3, 85.7)
- added REF**: DSUB-15-HD_Female_Horizontal_P2.29x1.98mm_EdgePinOffset8.35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, Connector_Dsub:DSUB-15-HD_Female_Horizontal_P2.29x1.98mm_EdgePinOffset8.35mm_Housed_MountingHolesOffset10.89mm, B.Cu at (127.4, 130.9)
- added REF**: DSUB-15-HD_Female_Horizontal_P2.29x1.98mm_EdgePinOffset8.35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, Connector_Dsub:DSUB-15-HD_Female_Horizontal_P2.29x1.98mm_EdgePinOffset8.35mm_Housed_MountingHolesOffset10.89mm, B.Cu at (166.0, 130.9)
