File: Schematics/Car LED Controller Schematic V9 - KiCAD/Car LED Controller Schematic V9 - KiCAD.kicad_sch (KiCad schematic)
At the start: 25 parts, among them J2 LCD, Relay, LED Signal, J3 5V Power In, J4 Reset Button, J4 Select Button, J4 ZSS-108-01-F-D-506, J5 DRL, Horn Sense, U1 ESP32-DEVKITC-32D, U2 BOB-12009, U3 PC817X3NSZ9F, U4 PC817X3NSZ9F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

Commit message: PCB and Schematic updates
Connections:
- net GND: no longer R1.2, R1.2, R1.2, U1.J2-4 (SENSOR_VN), U1.J2-5 (IO34), U1.J2-6 (IO35), U3.3, U4.3, U5.3
- net DRL Signal: now reaches C1.1, R4.1, R9.1, U1.J2-3 (SENSOR_VP)
- new net Horn: R1.2, U1.J2-4 (SENSOR_VN), U5.3
- new net L_Ind: R1.2, U1.J2-5 (IO34), U4.3
- new net R_Ind: R1.2, U1.J2-6 (IO35), U3.3
- no-connect marks 0 -> 9
Other:
- moved on the sheet: R1

Commit message: Update to schematic and PCBupdate
Parts:
- added D3: D_Schottky, Diode_THT:D_DO-41_SOD81_P10.16mm_Horizontal, symbol Device:D_Schottky
- added J7: DRL, Horn Sense, Connector_JST:JST_XH_B4B-XH-A_1x04_P2.50mm_Vertical, symbol Connector_Generic:Conn_01x04
- J2: value LCD, Relay, LED Signal -> LCD Display; footprint Connector_JST:JST_XH_B6B-XH-A_1x06_P2.50mm_Vertical -> Connector_JST:JST_XH_B4B-XH-A_1x04_P2.50mm_Vertical; symbol Connector_Generic:Conn_01x06 -> Connector_Generic:Conn_01x04
- J5: value DRL, Horn Sense -> DRL, Horn, Indicator; footprint Connector_JST:JST_XH_B6B-XH-A_1x06_P2.50mm_Vertical -> Connector_JST:JST_XH_B4B-XH-A_1x04_P2.50mm_Vertical; symbol Connector_Generic:Conn_01x06 -> Connector_Generic:Conn_01x04
Connections:
- net GND: now also J2.4 (Pin_4), D3.2 (A), J7.4 (GND); no longer J2.6 (GND), J4.04 (GND), J4.16 (GND), J5.6 (GND)
- net Horn: now also J5.3 (Horn), R4.1
- net LCD_1: now reaches J2.2 (Pin_2)
- net LCD_1: now also U2.HV3; no longer U2.HV1
- net LCD_2: now reaches J2.3 (Pin_3)
- net LCD_2: now also U2.HV4; no longer U2.HV2
- net DRL_L: now reaches D1.2 (A), J5.1 (DRL_L)
- net DRL_R: now reaches D2.2 (A), J5.2 (DRL_R)
- net IND_L: now reaches J5.4 (IND_L), R4.1
- net IND_R: now reaches R4.1
- net IND_R: now also J7.1 (IND_R); no longer J5.5 (R_Ind)
- new net: D3.1 (K), J4.04 (GND), J4.16 (GND)
- new net LED: J7.3 (LED), U2.HV2
- new net RELAY: J7.2 (Relay), U2.HV1
Other:
- moved on the sheet: J3

Commit message: updated pcb and schematic
Connections:
- net GND: now also D3.1 (K), J4.04 (GND), J4.16 (GND); no longer D3.2 (A), U1.J2-14 (GND1), U1.J3-1 (GND3), U1.J3-7 (GND2)
- net Horn: no longer R1.2, U1.J2-4 (SENSOR_VN), U5.3
- net L_Ind renamed L_Ind_Inp
- net R_Ind renamed R_Ind_Inp
- new net ESP32_GND: D3.2 (A), U1.J2-14 (GND1), U1.J3-1 (GND3), U1.J3-7 (GND2)
- new net Horn_Inp: R1.2, U1.J2-4 (SENSOR_VN), U5.3
Other:
- moved on the sheet: D3, J4

Commit message: PCB upload to manufacturing
Parts:
- D3: value D_Schottky -> 95SQ015
Changed lines of the file:
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@@
       (effects (font (size 1.27 1.27)))
     )
-    (property "Value" "D_Schottky" (at 101.6 172.72 0)
+    (property "Value" "95SQ015" (at 101.6 172.72 0)
       (effects (font (size 1.27 1.27)))
     )
@@
       (effects (font (size 1.27 1.27)) hide)
     )
-    (property "Datasheet" "~" (at 97.79 172.72 0)
+    (property "Datasheet" "https://www.smc-diodes.com/propdf/95SQ015%20N0181%20REV.A.pdf" (at 97.79 172.72 0)
       (effects (font (size 1.27 1.27)) hide)
     )
