File: Schematics/Car LED Controller Schematic V9 - KiCAD/Car LED Controller Schematic V9 - KiCAD.kicad_pcb (KiCad board)
At the start: 2 copper layers, 101.9 x 70 mm, 27 parts, among them J1 5V Power In, J2 Select Button, J3 LCD Display, J4 ZSS-108-01-F-D-506, J5 DRL, Horn, Indicator, J6 Reset Button, J7 DRL, Horn Sense, U1 ESP32-DEVKITC-32D, U2 BOB-12009, U3 PC817X3NSZ9F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

Commit message: updated pcb and schematic
Parts:
- moved D3 59.7 mm to (48.5, 30.7), turned to 0 degrees
- moved J1 9.29 mm to (46.3, 38.1), turned to 0 degrees
- moved J7 0.75 mm to (85.6, 58.9)
Connections:
- net /L_Ind renamed /L_Ind_Inp
- net /R_Ind renamed /R_Ind_Inp
- D3 pad 1: Net-(D3-K) -> GND
- D3 pad 2: GND -> /ESP32_GND
- J4 pad 04: Net-(D3-K) -> GND
- J4 pad 16: Net-(D3-K) -> GND
- R1 pad 2: /Horn -> /Horn_Inp
- U1 pad J2-14: GND -> /ESP32_GND
- U1 pad J2-4: /Horn -> /Horn_Inp
- U1 pad J3-1: GND -> /ESP32_GND
- U1 pad J3-7: GND -> /ESP32_GND
- U5 pad 3: /Horn -> /Horn_Inp
Routing:
- net /Horn_Inp: track 0.00 -> 90.3 mm, vias 0 -> 1
- net /Horn: track 99.8 -> 10.1 mm, vias 1 -> 0
- net /ESP32_GND: track 0.00 -> 65.9 mm
- net Net-(D3-K): track 31.5 -> 0.00 mm
- net +5V: track 202.9 -> 217.1 mm
- net +3.3V: track 100.4 -> 89.8 mm
- net Net-(J4-G1): track 87.2 -> 83.9 mm
- net Net-(J4-A): track 94.0 -> 91.2 mm
- net Net-(J2-Pin_1): track 73.9 -> 71.4 mm
- net /L_Ind_Inp: track 93.6 -> 94.8 mm
- net /DRL Signal: track 68.2 -> 67.1 mm
- net Net-(J4-E): track 88.8 -> 87.8 mm
- net Net-(J4-R2): track 85.2 -> 84.6 mm
- net /R_Ind_Inp: track 110.6 -> 111.2 mm
- net /LED: track 46.4 -> 45.9 mm
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
Commit message: PCB upload to manufacturing
Parts:
- moved J1 12.4 mm to (54.1, 28.4)
- moved D3 5.59 mm to (44.2, 34.3)
Routing:
- net GND: track 362.0 -> 368.9 mm
- net /ESP32_GND: track 65.9 -> 71.1 mm
- net +5V: track 217.1 -> 215.7 mm
- net +3.3V: track 89.8 -> 91.2 mm
Other:
- board text added: "LED Matrix Controller V9.1"
- board text removed: "LED Matrix Controller V9"

Commit message: PCB Update
Parts:
- moved D3 0.51 mm to (44.7, 34.3)
Routing:
- net Net-(D1-K): track 22.9 -> 24.6 mm
- net GND: track 368.9 -> 370.4 mm

Commit message: PCB Update
Parts:
- D3: footprint Diode_THT:D_DO-41_SOD81_P10.16mm_Horizontal -> Diode_THT:D_DO-201AD_P5.08mm_Vertical_AnodeUp
- moved D3 3.06 mm to (47.5, 35.6), turned to -90 degrees
Routing:
- net /ESP32_GND: track 71.3 -> 80.8 mm
- net +5V: track 215.7 -> 220.4 mm
- net GND: track 370.4 -> 369.1 mm
